Commit message: add gazebo stuff

File: urdf/kinova_kg3.urdf (robot description, URDF)
Before this commit: robot kinova_kg3, 9 links, 9 joints
Links:
- removed link jaco_link_finger_2_inner_1
- removed link jaco_link_finger_2_inner_2
Joints:
- removed joint jaco_joint_finger_2_inner_1
- removed joint jaco_joint_finger_2_inner_2
- removed joint jaco_joint_finger_2_innner_3

File: urdf/kinova_kg3.xacro (robot description, xacro)
@@ -1,6 +1,12 @@
 <?xml version="1.0"?>
-<robot name="kinova_kg3" xmlns:xacro="http://ros.org/wiki/xacro">
+<robot name="kinova_kg3"
+	xmlns:sensor="http://playerstage.sourceforge.net/gazebo/xmlschema/#sensor"
+    xmlns:controller="http://playerstage.sourceforge.net/gazebo/xmlschema/#controller"
+    xmlns:joint="http://playerstage.sourceforge.net/gazebo/xmlschema/#slider"
+	xmlns:interface="http://playerstage.sourceforge.net/gazebo/xmlschema/#interface"
+	xmlns:xacro="http://ros.org/wiki/xacro">
 	<property name="PKG" value="package://kinova_kg3/"/>
 	<property name="M_PI" value="3.14159265358979"/>
+	<xacro:include filename="kinova_kg3.gazebo.xacro"/>
 	<link name="jaco_link_hand">
 		<inertial>
@@ -31,4 +37,5 @@
 		</collision>
 	</link>
+	<xacro:kinova_kg3_gazebo />
 	<xacro:include filename="kinova_kg3_finger.xacro" />
 	<xacro:kinova_kg3_finger index="1" origin_xx="0.00228309324472738" origin_yy="-0.0312566848705875" origin_zz="0.114430431187145"

File: urdf/kinova_kg3_finger.xacro (robot description, xacro)
@@ -1,4 +1,5 @@
 <?xml version="1.0"?>
 <robot name="kinova_kg3_finger" xmlns:xacro="http://ros.org/wiki/xacro">
+	<xacro:include filename="kinova_kg3_finger.gazebo.xacro"/>
 	<xacro:macro name="kinova_kg3_finger" params="index origin_xx origin_yy origin_zz origin_r origin_p origin_y">
 		<joint name="jaco_joint_finger_${index}" type="revolute">
@@ -76,4 +77,5 @@
 			<axis xyz="0 0 1" />
 		</joint>
+		<xacro:kinova_kg3_finger_gazebo index="${index}" />
 	</xacro:macro>
 </robot>
