Commit message: add gazebo transmission things, add controllers

File: urdf/kinova_kg3.gazebo.xacro (robot description, xacro)
@@ -29,4 +29,9 @@
       </gripper>
     </gazebo>
+	<gazebo>
+		<plugin name="gazebo_ros_control" filename="libgazebo_ros_control.so">
+			<robotNamespace>kinova_kg3</robotNamespace>
+  		</plugin>
+    </gazebo>
   </xacro:macro>
 </robot>

File: urdf/kinova_kg3.urdf (robot description, URDF)
Before this commit: robot kinova_kg3, 7 links, 6 joints
Links:
- link jaco_link_finger_1: mass 0.00888493693152805 -> 0.05
- link jaco_link_finger_2: mass 0.00888493693152805 -> 0.05
- link jaco_link_finger_3: mass 0.00888493693152805 -> 0.05
- link jaco_link_finger_tip_1: mass 0.0124078189139213 -> 0.03
- link jaco_link_finger_tip_2: mass 0.0124078189139213 -> 0.03
- link jaco_link_finger_tip_3: mass 0.0124078189139213 -> 0.03
- link jaco_link_hand: mass 0.121634609410213 -> 0.49

File: urdf/kinova_kg3.xacro (robot description, xacro)
@@ -12,5 +12,5 @@
 		<inertial>
 		  <origin xyz="-0.000227690650068603 0.0042546911231965 0.0759513725294467" rpy="0 0 0" />
-		  <mass value="0.121634609410213" />
+		  <mass value="0.49" />
 		  <inertia
 			ixx="0.000215056800843909"

File: urdf/kinova_kg3_finger.xacro (robot description, xacro)
@@ -2,4 +2,5 @@
 <robot name="kinova_kg3_finger" xmlns:xacro="http://ros.org/wiki/xacro">
 	<xacro:include filename="kinova_kg3_finger.gazebo.xacro"/>
+	<xacro:include filename="kinova_kg3_finger.transmission.xacro"/>
 	<xacro:macro name="kinova_kg3_finger" params="index origin_xx origin_yy origin_zz origin_r origin_p origin_y">
 		<joint name="jaco_joint_finger_${index}" type="revolute">
@@ -16,5 +17,5 @@
 			rpy="0 0 0" />
 		  <mass
-			value="0.00888493693152805" />
+			value="0.05" />
 		  <inertia
 			ixx="1.04331946762797E-06"
@@ -47,5 +48,5 @@
 				rpy="0 0 0" />
 			  <mass
-				value="0.0124078189139213" />
+				value="0.03" />
 			  <inertia
 				ixx="6.8332629760199E-07"
@@ -78,4 +79,5 @@
 		</joint>
 		<xacro:kinova_kg3_finger_gazebo index="${index}" />
+		<xacro:kinova_kg3_finger_transmission index="${index}" />
 	</xacro:macro>
 </robot>
